File: hardware/buttons.sch (KiCad schematic (older format))
At the start: 52 parts, among them SW1 SW_Push, SW10 SW_Push, SW11 SW_Push, SW12 SW_Push, SW13 SW_Push, SW14 SW_Push, SW15 SW_Push, SW16 SW_Push, SW2 SW_Push, SW3 SW_Push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

Commit message: Dumb leds and stm32 magic
Parts:
- removed D17, D18, D19, D20, D21, D22, D23, D24, D25, D26, D27, D28, D29, D30, D31, D32: SK6812, LED_SMD:LED_SK6812_PLCC4_5.0x5.0mm_P3.2mm, symbol LED:SK6812
- SW10, SW12, SW14, SW16, SW2, SW6, SW8: footprint silicone_key_contact:silicone_key_contact -> silicone_key_contact:silicone_key_contact_mirrored
Connections:
- net labels removed: 5V, LEDS_IN
- wire segments 93 -> 60
- no-connect marks 1 -> 0

Commit message: Added lcsc partnumbers
Parts:
- D1, D10, D11, D12, D13, D14, D15, D16, D2, D3, D4, D5, D6, D7, D8, D9: LCSC (none) -> C81598
- R1, R2, R3, R4: LCSC (none) -> C25804
Changed lines of the file:
@@
 F 2 "Resistor_SMD:R_0603_1608Metric" V 2980 4400 50  0001 C CNN
 F 3 "~" H 3050 4400 50  0001 C CNN
+F 4 "C25804" H 3050 4400 50  0001 C CNN "LCSC"
 	1    3050 4400
 	1    0    0    -1
@@
 F 2 "Resistor_SMD:R_0603_1608Metric" V 4080 4400 50  0001 C CNN
 F 3 "~" H 4150 4400 50  0001 C CNN
+F 4 "C25804" H 4150 4400 50  0001 C CNN "LCSC"
 	1    4150 4400
 	1    0    0    -1
@@
 F 2 "Resistor_SMD:R_0603_1608Metric" V 5180 4400 50  0001 C CNN
 F 3 "~" H 5250 4400 50  0001 C CNN
+F 4 "C25804" H 5250 4400 50  0001 C CNN "LCSC"
 	1    5250 4400
 	1    0    0    -1
@@
 F 2 "Resistor_SMD:R_0603_1608Metric" V 6280 4400 50  0001 C CNN
 F 3 "~" H 6350 4400 50  0001 C CNN
+F 4 "C25804" H 6350 4400 50  0001 C CNN "LCSC"
 	1    6350 4400
 	1    0    0    -1
@@
 F 2 "Diode_SMD:D_SOD-123" H 2750 1625 50  0001 C CNN
 F 3 "https://www.vishay.com/docs/85748/1n4148w.pdf" H 2750 1800 50  0001 C CNN
+F 4 "C81598" H 2750 1800 50  0001 C CNN "LCSC"
 	1    2750 1800
 	-1   0    0    1
@@
 F 2 "Diode_SMD:D_SOD-123" H 3850 1625 50  0001 C CNN
 F 3 "https://www.vishay.com/docs/85748/1n4148w.pdf" H 3850 1800 50  0001 C CNN
+F 4 "C81598" H 3850 1800 50  0001 C CNN "LCSC"
 	1    3850 1800
 	-1   0    0    1
@@
 F 2 "Diode_SMD:D_SOD-123" H 4950 1625 50  0001 C CNN
 F 3 "https://www.vishay.com/docs/85748/1n4148w.pdf" H 4950 1800 50  0001 C CNN
+F 4 "C81598" H 4950 1800 50  0001 C CNN "LCSC"
 	1    4950 1800
 	-1   0    0    1
@@
 F 2 "Diode_SMD:D_SOD-123" H 6050 1625 50  0001 C CNN
 F 3 "https://www.vishay.com/docs/85748/1n4148w.pdf" H 6050 1800 50  0001 C CNN
+F 4 "C81598" H 6050 1800 50  0001 C CNN "LCSC"
 	1    6050 1800
 	-1   0    0    1
@@
 F 2 "Diode_SMD:D_SOD-123" H 2750 2325 50  0001 C CNN
 F 3 "https://www.vishay.com/docs/85748/1n4148w.pdf" H 2750 2500 50  0001 C CNN
+F 4 "C81598" H 2750 2500 50  0001 C CNN "LCSC"
 	1    2750 2500
 	-1   0    0    1
@@
 F 2 "Diode_SMD:D_SOD-123" H 3850 2325 50  0001 C CNN
 F 3 "https://www.vishay.com/docs/85748/1n4148w.pdf" H 3850 2500 50  0001 C CNN
+F 4 "C81598" H 3850 2500 50  0001 C CNN "LCSC"
 	1    3850 2500
 	-1   0    0    1
@@
 F 2 "Diode_SMD:D_SOD-123" H 4950 2325 50  0001 C CNN
 F 3 "https://www.vishay.com/docs/85748/1n4148w.pdf" H 4950 2500 50  0001 C CNN
+F 4 "C81598" H 4950 2500 50  0001 C CNN "LCSC"
 	1    4950 2500
 	-1   0    0    1
@@
 F 2 "Diode_SMD:D_SOD-123" H 6050 2325 50  0001 C CNN
 F 3 "https://www.vishay.com/docs/85748/1n4148w.pdf" H 6050 2500 50  0001 C CNN
+F 4 "C81598" H 6050 2500 50  0001 C CNN "LCSC"
 	1    6050 2500
 	-1   0    0    1
@@
 F 2 "Diode_SMD:D_SOD-123" H 2750 3025 50  0001 C CNN
 F 3 "https://www.vishay.com/docs/85748/1n4148w.pdf" H 2750 3200 50  0001 C CNN
+F 4 "C81598" H 2750 3200 50  0001 C CNN "LCSC"
 	1    2750 3200
 	-1   0    0    1
@@
 F 2 "Diode_SMD:D_SOD-123" H 3850 3025 50  0001 C CNN
 F 3 "https://www.vishay.com/docs/85748/1n4148w.pdf" H 3850 3200 50  0001 C CNN
+F 4 "C81598" H 3850 3200 50  0001 C CNN "LCSC"
 	1    3850 3200
 	-1   0    0    1
@@
 F 2 "Diode_SMD:D_SOD-123" H 4950 3025 50  0001 C CNN
 F 3 "https://www.vishay.com/docs/85748/1n4148w.pdf" H 4950 3200 50  0001 C CNN
+F 4 "C81598" H 4950 3200 50  0001 C CNN "LCSC"
 	1    4950 3200
 	-1   0    0    1
@@
 F 2 "Diode_SMD:D_SOD-123" H 6050 3025 50  0001 C CNN
 F 3 "https://www.vishay.com/docs/85748/1n4148w.pdf" H 6050 3200 50  0001 C CNN
+F 4 "C81598" H 6050 3200 50  0001 C CNN "LCSC"
 	1    6050 3200
 	-1   0    0    1
@@
 F 2 "Diode_SMD:D_SOD-123" H 2750 3725 50  0001 C CNN
 F 3 "https://www.vishay.com/docs/85748/1n4148w.pdf" H 2750 3900 50  0001 C CNN
+F 4 "C81598" H 2750 3900 50  0001 C CNN "LCSC"
 	1    2750 3900
 	-1   0    0    1
@@
 F 2 "Diode_SMD:D_SOD-123" H 3850 3725 50  0001 C CNN
 F 3 "https://www.vishay.com/docs/85748/1n4148w.pdf" H 3850 3900 50  0001 C CNN
+F 4 "C81598" H 3850 3900 50  0001 C CNN "LCSC"
 	1    3850 3900
 	-1   0    0    1
@@
 F 2 "Diode_SMD:D_SOD-123" H 4950 3725 50  0001 C CNN
 F 3 "https://www.vishay.com/docs/85748/1n4148w.pdf" H 4950 3900 50  0001 C CNN
+F 4 "C81598" H 4950 3900 50  0001 C CNN "LCSC"
 	1    4950 3900
 	-1   0    0    1
@@
 F 2 "Diode_SMD:D_SOD-123" H 6050 3725 50  0001 C CNN
 F 3 "https://www.vishay.com/docs/85748/1n4148w.pdf" H 6050 3900 50  0001 C CNN
+F 4 "C81598" H 6050 3900 50  0001 C CNN "LCSC"
 	1    6050 3900
 	-1   0    0    1
