File: hardware/led_matrix.sch (KiCad schematic (older format))
At the start: 25 parts, among them U10 SM16106, U11 SM16106, U9 SM16106

Commit message: Updated lcsc part numbers
Parts:
- R11, R26, R6: LCSC (none) -> C23241
Changed lines of the file:
@@
 F 2 "Resistor_SMD:R_0603_1608Metric" V 8680 5150 50  0001 C CNN
 F 3 "~" H 8750 5150 50  0001 C CNN
-F 4 "" H 8750 5150 50  0001 C CNN "LCSC"
+F 4 "C23241" H 8750 5150 50  0001 C CNN "LCSC"
 	1    8750 5150
 	1    0    0    -1
@@
 F 2 "Resistor_SMD:R_0603_1608Metric" V 8630 3700 50  0001 C CNN
 F 3 "~" H 8700 3700 50  0001 C CNN
-F 4 "" H 8700 3700 50  0001 C CNN "LCSC"
+F 4 "C23241" H 8700 3700 50  0001 C CNN "LCSC"
 	1    8700 3700
 	1    0    0    -1
@@
 F 2 "Resistor_SMD:R_0603_1608Metric" V 8630 2250 50  0001 C CNN
 F 3 "~" H 8700 2250 50  0001 C CNN
-F 4 "" H 8700 2250 50  0001 C CNN "LCSC"
+F 4 "C23241" H 8700 2250 50  0001 C CNN "LCSC"
 	1    8700 2250
 	1    0    0    -1

Commit message: Gerber files for v1
Connections:
- no-connect marks 0 -> 1
Changed lines of the file:
@@
 Wire Wire Line
 	9250 5350 9250 5200
+NoConn ~ 8150 5100
 Wire Bus Line
 	3050 1800 6150 1800
